File: hardware/can_datalogger_board/untitled.kicad_sch (KiCad schematic)
At the start: 36 parts, among them SW1 JS202011SCQN, SW2 JS202011SCQN, U2 MCP2515T-I/ML, U3 MCP2515T-I/ML, U4 TCAN3403DRQ1, U5 TCAN3403DRQ1, Y1 20 MHz, Y2 20 MHz

Commit message: PCB component placement
Parts:
- U2, U3: footprint Package_SO:SOIC-18W_7.5x11.6mm_P1.27mm -> Package_DFN_QFN:QFN-20-1EP_4x4mm_P0.5mm_EP2.5x2.5mm
Changed lines of the file:
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@@
 			)
 		)
-		(property "Footprint" "Package_SO:SOIC-18W_7.5x11.6mm_P1.27mm"
+		(property "Footprint" "Package_DFN_QFN:QFN-20-1EP_4x4mm_P0.5mm_EP2.5x2.5mm"
 			(at 78.74 170.18 0)
 			(effects
@@
 			)
 		)
-		(property "Footprint" "Package_SO:SOIC-18W_7.5x11.6mm_P1.27mm"
+		(property "Footprint" "Package_DFN_QFN:QFN-20-1EP_4x4mm_P0.5mm_EP2.5x2.5mm"
 			(at 78.74 91.44 0)
 			(effects
